File: pcb/usb.kicad_sch (KiCad schematic)
At the start: 6 parts, among them J2 USB_C_Receptacle_USB2.0_14P, U5 CP2102N-Axx-xQFN24

Commit message: Protection
Parts:
- added FL1: ECMF02-4CMX8, ECMF02-4CMX8:FIL_ECMF02-4CMX8, symbol ECMF02-4CMX8:ECMF02-4CMX8
Connections:
- net D+: now also FL1.6 (D+_6); no longer J2.A6 (D+), J2.B6 (D+)
- net D-: now also FL1.7 (D-_7); no longer J2.A7 (D-), J2.B7 (D-)
- net GND: now also FL1.5 (GND_5), FL1.8 (GND_8)
- net VBUS: now also FL1.1 (VBUS)
- new net: FL1.3 (D+_3), J2.A6 (D+), J2.B6 (D+)
- new net: FL1.2 (D-_2), J2.A7 (D-), J2.B7 (D-)
Other:
- note removed: "Add USB<->Ser"
- note removed: "TODO: Add protection"
- note removed: "TODO: is this back-powered when USB not connected?"
- moved on the sheet: J2
